File: Fan controller schematics/LED control.sch (KiCad schematic (older format))
At the start: 53 parts, among them U1 ULN2003A, U10 74HC595, U11 74HC595, U12 ULN2003A, U13 ULN2003A, U2 74HC595, U3 ULN2003A, U4 74HC595, U5 ULN2003A, U6 74HC595, U7 ULN2003A, U8 74HC595, U9 ULN2003A

Commit message: Add ADC filter and ref
Parts:
- renumbered R12 to R10, R13 to R11, R14 to R12, R15 to R13, R16 to R14, R17 to R15, R18 to R16, R19 to R17, R20 to R18, R21 to R19, R22 to R20, R23 to R21, R24 to R22, R25 to R23, R26 to R24, R27 to R25, R28 to R26, R29 to R27, R10 to R8, R11 to R9, U9 to U10, U10 to U11, U11 to U12, U12 to U13, U13 to U14, U1 to U2, U2 to U3, U3 to U4, U4 to U5, U5 to U6, U6 to U7, U7 to U8, U8 to U9

Commit message: Update schematic to v1.3
Parts:
- removed D16, D17, D18, D19, D20, D21, D22, D23, D24, D25: RED 5mm LED, symbol LED
- removed R18, R19, R20, R21, R22, R23, R24, R25, R26, R27: 200, symbol R
- removed U11, U12: 74HC595, symbol 74HC595
- removed U13, U14: ULN2003A, symbol ULN2003A
- renumbered D9 to D10, D10 to D11, D11 to D12, D12 to D13, D13 to D14, D14 to D15, D15 to D16, D6 to D7, D7 to D8, D8 to D9, R9 to R10, R10 to R11, R11 to R12, R12 to R13, R13 to R14, R14 to R15, R15 to R16, R16 to R17, R17 to R18, R8 to R9
Connections:
- no-connect marks 0 -> 14
